Commit message: continuação aps 2

File: src/rm_description/urdf/differential_robot.xacro (robot description, xacro)
@@ -65,24 +65,49 @@
   </joint>
   <!-- ===================== -->
-  <!-- CASTER BALL           -->
+  <!-- CASTER BALLS          -->
   <!-- ===================== -->
-  <xacro:property name="caster_radius" value="0.02"/>
-  <link name="caster_ball">
+  <xacro:property name="caster_radius" value="0.025"/>
+  <link name="front_caster_ball">
     <visual>
       <origin xyz="0 0 0" rpy="0 0 0"/>
-      <geometry><sphere radius="${caster_radius}"/></geometry>
+      <geometry>
+        <sphere radius="${caster_radius}"/>
+      </geometry>
     </visual>
     <collision>
       <origin xyz="0 0 0" rpy="0 0 0"/>
-      <geometry><sphere radius="${caster_radius}"/></geometry>
+      <geometry>
+        <sphere radius="${caster_radius}"/>
+      </geometry>
     </collision>
-    <xacro:inertial_sphere mass="0.2" radius="${caster_radius}">
+    <xacro:inertial_sphere mass="0.03" radius="${caster_radius}">
       <origin xyz="0 0 0" rpy="0 0 0"/>
     </xacro:inertial_sphere>
   </link>
-  <joint name="caster_joint" type="fixed">
+  <joint name="front_caster_joint" type="fixed">
     <parent link="base_link"/>
-    <child link="caster_ball"/>
-    <!-- z = -wheel_radius + caster_radius -> toca o chão -->
+    <child link="front_caster_ball"/>
+    <origin xyz="0.12 0 ${-wheel_radius + caster_radius}" rpy="0 0 0"/>
+  </joint>
+  <link name="rear_caster_ball">
+    <visual>
+      <origin xyz="0 0 0" rpy="0 0 0"/>
+      <geometry>
+        <sphere radius="${caster_radius}"/>
+      </geometry>
+    </visual>
+    <collision>
+      <origin xyz="0 0 0" rpy="0 0 0"/>
+      <geometry>
+        <sphere radius="${caster_radius}"/>
+      </geometry>
+    </collision>
+    <xacro:inertial_sphere mass="0.03" radius="${caster_radius}">
+      <origin xyz="0 0 0" rpy="0 0 0"/>
+    </xacro:inertial_sphere>
+  </link>
+  <joint name="rear_caster_joint" type="fixed">
+    <parent link="base_link"/>
+    <child link="rear_caster_ball"/>
     <origin xyz="-0.12 0 ${-wheel_radius + caster_radius}" rpy="0 0 0"/>
   </joint>
@@ -104,9 +129,13 @@
     <visual>
       <origin xyz="0 0 0" rpy="0 0 0"/>
-      <geometry><cylinder radius="${lidar_radius}" length="${lidar_height}"/></geometry>
+      <geometry>
+        <cylinder radius="${lidar_radius}" length="${lidar_height}"/>
+      </geometry>
     </visual>
     <collision>
       <origin xyz="0 0 0" rpy="0 0 0"/>
-      <geometry><cylinder radius="${lidar_radius}" length="${lidar_height}"/></geometry>
+      <geometry>
+        <cylinder radius="${lidar_radius}" length="${lidar_height}"/>
+      </geometry>
     </collision>
     <xacro:inertial_cylinder mass="0.2" length="${lidar_height}" radius="${lidar_radius}">
@@ -125,9 +154,13 @@
     <visual>
       <origin xyz="0 0 0" rpy="0 0 0"/>
-      <geometry><box size="0.04 0.04 0.02"/></geometry>
+      <geometry>
+        <box size="0.04 0.04 0.02"/>
+      </geometry>
     </visual>
     <collision>
       <origin xyz="0 0 0" rpy="0 0 0"/>
-      <geometry><box size="0.04 0.04 0.02"/></geometry>
+      <geometry>
+        <box size="0.04 0.04 0.02"/>
+      </geometry>
     </collision>
     <xacro:inertial_box mass="0.1" x="0.04" y="0.04" z="0.02">
